File: 6_Test/2_PCB/test_board/schematics/AnalogSupply/analogSupply_final.kicad_sch (KiCad schematic)
At the start: 17 parts

Commit message: Adjusted Edits 11_25_24
Parts:
- C? (x4): footprint CAP_CL05_SAM -> cap100nFFootprints:CAP_CL05_SAM
- C? (x3): footprint CAP_0603_CL10A_1P6XP8_SAM -> Cap4.7uFFootprints:CAP_0603_CL10A_1P6XP8_SAM
- L?: footprint IND_BLM18_0603_MUR -> ferriteBead120OhmFootprints:IND_BLM18_0603_MUR
- R?: value 4.7k -> 1k
- R? (x3): footprint PV37W103C01B00:TRIM_PV37W103C01B00 -> ECE628_lib:potentiometer_10turn
- U?: value LDO_Analog_Supply -> TPS74501PDRVR; footprint DRV0006A -> tps745Footprints:DRV0006A
Connections:
- net AVSS: now also C?.1, C?.2
- net GND: no longer C?.1, C?.2
- net at R?.2: now also R?.2, U?.2 (FB); no longer R?.3
Other:
- moved on the sheet: C?, L?, R?
