File: 6_Test/2_PCB/test_board/schematics/Buffer/buffer_final.kicad_sch (KiCad schematic)
At the start: 15 parts, among them U1 SN74ALVCH162827DLR

Commit message: Adjusted Edits 11_25_24
Parts:
- added C23, C25, C27, C29: 4.7u, Capacitor_SMD:C_0603_1608Metric, symbol Device:C
- added C24, C26, C28, C30: 100n, Capacitor_SMD:C_0402_1005Metric, symbol Device:C
- added J11: Buffer_PWR_Jumper, symbol Connector:Conn_01x02_Pin
- U1: footprint DL56 -> 74ALVCHFootprints:DL56
- renumbered R31 to R28, R32 to R29
Connections:
- net GND: now also C23.2, C24.2, C25.2, C26.2, C27.2, C28.2, C29.2, C30.2; no longer U1.20 (2Y5), U1.21 (2Y6), U1.23 (2Y7), U1.24 (2Y8), U1.26 (2Y9), U1.27 (2Y10)
- net VCC: now also C23.1, C24.1, C25.1, C26.1, C27.1, C28.1, C29.1, C30.1, J11.1 (Pin_1), J11.2 (Pin_2)
Other:
- moved on the sheet: R1, R10, R11, R12, R2, R28, R29, R3, R4, R5, R6, R7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
