File: 6_Test/2_PCB/test_board/schematics/LDOCircuitry/LDO_circuitry_final.kicad_sch (KiCad schematic)
At the start: 6 parts

Commit message: Adjusted Edits 11_25_24
Parts:
- R?: footprint POT_PV37W_MUR -> ECE628_lib:potentiometer_10turn
Changed lines of the file:
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@@
 		(dnp no)
 		(property "Reference" "C?"
-			(at 143.764 111.506 0)
+			(at 143.002 109.22 0)
 			(effects
 				(font
@@
 		)
 		(property "Value" "4.7uF"
-			(at 144.018 109.474 0)
+			(at 143.51 111.252 0)
 			(effects
 				(font
@@
 			(project "board_main"
 				(path "/9c0580c5-7bd5-4e54-bf4c-826aa4ac3630/104c40d7-ae25-447b-8675-a765b7f78bca"
-					(reference "C8")
+					(reference "C37")
 					(unit 1)
 				)
@@
 			(project "board_main"
 				(path "/9c0580c5-7bd5-4e54-bf4c-826aa4ac3630/104c40d7-ae25-447b-8675-a765b7f78bca"
-					(reference "R7")
+					(reference "R30")
 					(unit 1)
 				)
@@
 		(dnp no)
 		(property "Reference" "C?"
-			(at 155.448 111.506 0)
+			(at 154.94 109.474 0)
 			(effects
 				(font
@@
 		)
 		(property "Value" "100nF"
-			(at 155.702 109.474 0)
+			(at 155.194 111.252 0)
 			(effects
 				(font
@@
 			(project "board_main"
 				(path "/9c0580c5-7bd5-4e54-bf4c-826aa4ac3630/104c40d7-ae25-447b-8675-a765b7f78bca"
-					(reference "C9")
+					(reference "C38")
 					(unit 1)
 				)
@@
 			(project "board_main"
 				(path "/9c0580c5-7bd5-4e54-bf4c-826aa4ac3630/104c40d7-ae25-447b-8675-a765b7f78bca"
-					(reference "C7")
+					(reference "C36")
 					(unit 1)
 				)
@@
 			)
 		)
-		(property "Footprint" "POT_PV37W_MUR"
+		(property "Footprint" "ECE628_lib:potentiometer_10turn"
 			(at 114.3 105.41 0)
 			(effects
@@
 			(project "board_main"
 				(path "/9c0580c5-7bd5-4e54-bf4c-826aa4ac3630/104c40d7-ae25-447b-8675-a765b7f78bca"
-					(reference "R8")
+					(reference "R31")
 					(unit 1)
 				)
@@
 			(project "board_main"
 				(path "/9c0580c5-7bd5-4e54-bf4c-826aa4ac3630/104c40d7-ae25-447b-8675-a765b7f78bca"
-					(reference "R9")
-					(unit 1)
-				)
+					(reference "R32")
+					(unit 1)
+				)
